Commit message: add kalman filter to stablize the output detection

File: src/forklift_simulator/urdf/RX20_16/base.xacro (robot description, xacro)
@@ -6,6 +6,6 @@
    <inertial>
     <origin xyz="-0.8 0 0.417" rpy="0 0 0"/>
-     <xacro:box_inertia mass="50" x="1.843" y="1.1" z="0.835"/>
-    <mass value= "50"/>
+     <xacro:box_inertia mass="10" x="1.843" y="1.1" z="0.835"/>
+    <mass value= "10"/>
     </inertial>
     <collision>

File: src/forklift_simulator/urdf/RX20_16/d435_sensor.xacro (robot description, xacro)
@@ -43,5 +43,5 @@
         <always_on>1</always_on>
         <update_rate>30</update_rate>
-        <visualize>1</visualize>
+        <visualize>0</visualize>
       </sensor>
       <sensor name="${camera_name}ired1" type="camera">

File: src/forklift_simulator/urdf/RX20_16/front_wheels.xacro (robot description, xacro)
@@ -30,5 +30,5 @@
      <dynamics damping="0.01" friction="1.0"/>
   </joint>
-   <!-- <transmission name="trans_dynamic_${name}">
+   <transmission name="trans_dynamic_${name}">
     <type>transmission_interface/SimpleTransmission</type>
     <joint name="wheel_${name}_driving_joint">
@@ -39,11 +39,12 @@
       <mechanicalReduction>1</mechanicalReduction>
     </actuator>
-  </transmission> -->
+  </transmission>
   <gazebo reference="wheel_${name}_driving_link">
 			<mu1>1.0</mu1>
 			<mu2>1.0</mu2>
-			<kp>10000000.0</kp>
+			<!-- <kp>10000000.0</kp> -->
+			<kp>1000000000.0</kp>
 			<kd>1000.0</kd>
-			<minDepth>0.005</minDepth>
+			<minDepth>0.002</minDepth>
 			<maxVel>0</maxVel>
 		</gazebo>

File: src/forklift_simulator/urdf/RX20_16/lib_ackermansteer.xacro (robot description, xacro)
@@ -9,11 +9,12 @@
          <publishWheelTF>false</publishWheelTF>
          <publishOdomTF>true</publishOdomTF>
-         <wheelDiameter>0.36</wheelDiameter>
+         <driveWheelDiameter>0.36</driveWheelDiameter>
          <wheelAcceleration>0.0</wheelAcceleration>
-         <wheelTorque>50.0</wheelTorque>
+         <wheelTorque>500.0</wheelTorque>
          <updateRate>50.0</updateRate>
          <!-- Wheel Placement -->
          <wheelbase>1.429</wheelbase>
-         <wheelSeparation>0.932</wheelSeparation>
+         <steerWheelSeparation>0.932</steerWheelSeparation>
+         <driveWheelSeparation>0.808</driveWheelSeparation>
          <!-- Wheel Joints -->
          <RR_driveJoint>wheel_right_driving_joint</RR_driveJoint>
@@ -29,18 +30,22 @@
          - - - - - - - - - - - - - - - - - - - - - - - - - -  -->
          <!-- Wheel Velocity PID settings -->
-         <drive_p>500.0</drive_p>
+         <drive_p>200.0</drive_p>
          <drive_i>0.0</drive_i>
          <drive_d>0.0</drive_d>
          <drive_imax>1.0</drive_imax>
          <drive_imin>-1.0</drive_imin>
-         <drive_max_effort>200.0</drive_max_effort>
+         <drive_max_effort>500.0</drive_max_effort>
          <!-- Steering PID settings -->
-         <steer_p>100.0</steer_p>
+         <steer_p>300.0</steer_p>
          <steer_i>0.0</steer_i>
-         <steer_d>1.0</steer_d>
+         <steer_d>0.0</steer_d>
          <steer_imax>5.0</steer_imax>
          <steer_imin>-5.0</steer_imin>
          <steer_max_effort>600.0</steer_max_effort>
          <steer_init_angle>0.0</steer_init_angle>
+         <publishWheelJointState>true</publishWheelJointState>
+         <drive_init_velocity>0.0</drive_init_velocity>
+         <back_flip_model>true</back_flip_model>
+         <safety_threshold_drive_vel>100.0</safety_threshold_drive_vel>
       </plugin>
     </gazebo>

File: src/forklift_simulator/urdf/RX20_16/loading_forklift_joints.xacro (robot description, xacro)
@@ -50,5 +50,5 @@
     <origin xyz="0.134 0 0.22" rpy="0 0 0" />
     <axis xyz="0 0 1" />
-    <limit lower="0.05" upper="2" effort="100" velocity="0.3"/>
+    <limit lower="-0.2" upper="2" effort="100" velocity="0.3"/>
      <dynamics damping="100.0" friction="1"/>
   </joint>
@@ -115,21 +115,57 @@
     </plugin>
   </gazebo>
-  <!-- <link name='box'>
+  <link name='box1'>
     <collision>
       <geometry>
-        <box size="1.2 0.8 0.1"/>
+        <box size="0.8 0.08 0.042"/>
       </geometry>
     </collision>
-    <visual>
+    <!-- <visual>
       <geometry>
-        <box size="1.2 0.8 0.1"/>
+        <box size="0.8 0.08 0.04"/>
       </geometry>
-    </visual>
+    </visual> -->
+  </link>
+  <joint name="pad_joint1" type="fixed">
+    <parent link="sideshift_link" />
+    <child link="box1" />
+    <origin xyz="0.4 0.189 0.02" rpy="0 0 0" />
+    <axis xyz="0 0 1" />
+  </joint>
+  <link name='box2'>
+    <collision>
+      <geometry>
+        <box size="0.8 0.08 0.042"/>
+      </geometry>
+    </collision>
+    <!-- <visual>
+      <geometry>
+        <box size="0.8 0.08 0.04"/>
+      </geometry>
+    </visual> -->
+  </link>
+  <joint name="pad_joint2" type="fixed">
+    <parent link="sideshift_link" />
+    <child link="box2" />
+    <origin xyz="0.4 -0.189 0.02" rpy="0 0 0" />
+    <axis xyz="0 0 1" />
+  </joint>
+  <link name='box'>
+    <collision>
+      <geometry>
+        <box size="0.02 0.2 0.1"/>
+      </geometry>
+    </collision>
+    <!-- <visual>
+      <geometry>
+        <box size="0.02 0.2 0.1"/>
+      </geometry>
+    </visual> -->
   </link>
   <joint name="pad_joint" type="fixed">
-    <parent link="tilt_link" />
+    <parent link="sideshift_link" />
     <child link="box" />
-    <origin xyz="0.7 0 0.06" rpy="0 0 0" />
+    <origin xyz="0.0 0.0 0.05" rpy="0 0 0" />
     <axis xyz="0 0 1" />
-  </joint> -->
+  </joint>
   </robot>

File: src/forklift_simulator/urdf/RX20_16/main.xacro (robot description, xacro)
@@ -10,11 +10,12 @@
 <xacro:include filename="$(find forklift_simulator)/urdf/RX20_16/loading_forklift_joints.xacro" />
 <xacro:include filename="$(find forklift_simulator)/urdf/RX20_16/lib_ackermansteer.xacro" />
-<xacro:camera_d435 name="camera" topics_ns="camera" parent="base_link"
-    publish_pointcloud="true"> <origin xyz="0.35 0 0.4" rpy="0 0.0 0" /> </xacro:camera_d435>
+<xacro:camera_d435 name="camera" topics_ns="camera" parent="lift_link" publish_pointcloud="true"> <origin xyz="0.02 0 0.1" rpy="0 0 0" /> </xacro:camera_d435>
 <xacro:rx20_steer_wheel name="left" x_steering="-1.429" y_steering="0.404" z_steering="0.06" radius="0.150" width="0.15" flip="-1" />
 <xacro:rx20_steer_wheel name="right" x_steering="-1.429" y_steering="-0.404" z_steering="0.06" radius="0.150" width="0.15" flip="-1" />
 <xacro:rx20_front_wheel name="right" x_loading="0.0" y_loading="0.466" z_loading="0.0" radius="0.18" width="0.18" flip="-1" />
 <xacro:rx20_front_wheel name="left" x_loading="0.0" y_loading="-0.466" z_loading="0.0" radius="0.18" width="0.18" flip="-1" />
-<xacro:nav_lidar name="one"  x="0.211"  y="-0.6" z="0.15" roll="0" pitch="0" yaw="1.57" resolution="1"/>
+<!-- <xacro:nav_lidar name="one"  x="0.5"  y="0.0" z="1.8" roll="0" pitch="0" yaw="0.0" resolution="1"/> -->
+<!-- <xacro:detection_lidar name="front"  x="0.0"  y="0.0" z="2.0" roll="0" pitch="0" yaw="0" resolution="1"/> -->
+<xacro:nav_lidar name="back"  x="0.2"  y="-0.6" z="-0.1" roll="0" pitch="0" yaw="1.57" resolution="1"/>
 <!-- <xacro:nav_lidar name="front"  x="0"  y="0.4" z="0.1" roll="0" pitch="0" yaw="-1.57" resolution="1"/> -->
 <!-- <xacro:detection_lidar name="front"  x="0.0"  y="0.0" z="0.6" roll="0" pitch="0" yaw="0" resolution="1"/> -->

File: src/forklift_simulator/urdf/RX20_16/nav_lidar.xacro (robot description, xacro)
@@ -29,9 +29,15 @@
           <scan>
             <horizontal>
-              <samples>270</samples>
+              <samples>1440</samples>
                 <resolution>1</resolution>
               <min_angle>0</min_angle>
-                <max_angle>4.71238</max_angle>
+                <max_angle>6.28</max_angle>
             </horizontal>
+            <!-- <vertical>
+              <samples>10</samples>
+                <resolution>1</resolution>
+              <min_angle>-0.5</min_angle>
+                <max_angle>0.5</max_angle>
+            </vertical> -->
           </scan>
             <range>

File: src/forklift_simulator/urdf/RX20_16/steer_wheels.xacro (robot description, xacro)
@@ -57,7 +57,7 @@
     <!-- <joint_properties damping="1.0" friction="0.3"/> -->
         <limit effort="100" velocity="100"/>
-     <dynamics damping="0.01" friction="1.0"/>
+     <dynamics damping="0.01" friction="0.0"/>
   </joint>
-  <!-- <transmission name="trans_steering_${name}">
+  <transmission name="trans_steering_${name}">
     <type>transmission_interface/SimpleTransmission</type>
     <joint name="wheel_${name}_steering_joint">
@@ -68,5 +68,5 @@
       <mechanicalReduction>1</mechanicalReduction>
     </actuator>
-  </transmission> -->
+  </transmission>
   <!-- <transmission name="trans_dynamic_${name}">
     <type>transmission_interface/SimpleTransmission</type>
@@ -82,7 +82,8 @@
 			<mu1>1</mu1>
 			<mu2>1</mu2>
-			<kp>10000000.0</kp>
+			<!-- <kp>10000000.0</kp> -->
+			<kp>1000000000.0</kp>
 			<kd>1000.0</kd>
-			<minDepth>0.005</minDepth>
+			<minDepth>0.002</minDepth>
 			<maxVel>0</maxVel>
 		</gazebo>
